File: bitcrane.kicad_sch (KiCad schematic)
At the start: 113 parts, among them J1 PSU Comm, J11 USB_C_Receptacle_USB2.0, J12 0455580003, J13 2x9P 2mm, J14 0353180420, J15 0353180420, J16 0353180420, J17 0353180420, J3 61900411021, J4 61900411021, Q1 DMP3013SFV-7, U1 FT4232HQ, U2 RT9080-33GJ5, U3 M93C46-WDW6TP, U5 EMC2305, Y1 12MHz

Commit message: switch schematic to RP2350. PCB not updated yet
Parts:
- removed C1, C2: 27pf, Capacitor_SMD:C_0805_2012Metric, symbol Device:C
- removed C18, C21: 4.7uF, Capacitor_SMD:C_0805_2012Metric, symbol Device:C
- removed C6: 3.3uF, Capacitor_SMD:C_0805_2012Metric, symbol Device:C
- removed FB1, FB2: FerriteBead_Small, Resistor_SMD:R_0603_1608Metric, symbol Device:FerriteBead_Small
- removed J11: USB_C_Receptacle_USB2.0, bitcrane:USB-C-SMD_G-SWITCH_GT-USB-7010ASV, symbol bitcrane:GT-USB-7010ASV
- removed R11: 1k, Resistor_SMD:R_0805_2012Metric, symbol Device:R_US
- removed R12: 12k, Resistor_SMD:R_0805_2012Metric, symbol Device:R_US
- removed R28 (x2): 4.7k, Resistor_SMD:R_0805_2012Metric, symbol Device:R_US
- removed R4, R5: 5.1k, Resistor_SMD:R_0805_2012Metric, symbol Device:R_US
- removed R6: 2.2k, Resistor_SMD:R_0805_2012Metric, symbol Device:R_US
- removed R7, R8, R9: 10k, Resistor_SMD:R_0805_2012Metric, symbol Device:R_US
- removed TP6 (x21): TestPoint, TestPoint:TestPoint_Pad_D1.5mm, symbol Connector:TestPoint
- removed U1: FT4232HQ, bitcrane:QFN50P900X900X105-65N, symbol bitcrane:FT4232HQ-REEL
- removed U3: M93C46-WDW6TP, bitcrane:TSSOP-8_L4.4-W3.0-P0.65-LS6.4-BL, symbol bitcrane:M93C46-WDW6TP
- removed Y1: 12MHz, Crystal:Crystal_SMD_3225-4Pin_3.2x2.5mm, symbol bitcrane:405C35B12M00000
- added C14, C15, C18, C20, C22, C24, C26: 4.7u, Capacitor_SMD:C_0402_1005Metric, symbol UPduino_v3.0:Device_C
- added C19, C21, C23, C25, C27, C28, C29, C30, C31, C32, C33: 0.1u, Capacitor_SMD:C_0402_1005Metric, symbol UPduino_v3.0:Device_C
- added D2, D3: 1N5819WS, Diode_SMD:D_SOD-323, symbol Device:D_Schottky
- added J14: USB_C_Receptacle_USB2.0, Connector_USB:USB_C_Receptacle_HRO_TYPE-C-31-M-12, symbol Connector:USB_C_Receptacle_USB2.0
- added J15: BM03B-SRSS-TB, Connector_JST:JST_SH_BM03B-SRSS-TB_1x03-1MP_P1.00mm_Vertical, symbol Connector_Generic_MountingPin:Conn_01x03_MountingPin
- added L1: 3.3u, RP2350_60QFN_minimal:L_pol_2016, symbol Device:L
- added PTC1: MF-FSMF035X-2, Resistor_SMD:R_0603_1608Metric, symbol Device:R_US
- added R31, R37, R38: 27, Resistor_SMD:R_0402_1005Metric, symbol Device:R_US
- added R32, R34: 1k, Resistor_SMD:R_0402_1005Metric, symbol Device:R_US
- added R33: 10k, Resistor_SMD:R_0402_1005Metric, symbol Device:R_US
- added R35: 10K, Resistor_SMD:R_0402_1005Metric, symbol Device:R_US
- added R36: 100, Resistor_SMD:R_0402_1005Metric, symbol Device:R_US
- added SW1: CS1213AGF260, CUSTOM:PTS820J25KSMTRLFS, symbol Switch:SW_Push
- added U3: RP2350_80QFN, RP2350_60QFN_minimal:RP2350B_QFN-80_EP_10.573x10.573_Pitch0.4mm, symbol MCU_RaspberryPi_RP2350:RP2350_80QFN
- added U4: W25Q32JVSSIQ, Package_SO:SOIC-8_5.23x5.23mm_P1.27mm, symbol UPduino_v3.0:W25Q32JVSS-Memory_Flash
- added Y1: ABM8-272-T3, Crystal:Crystal_SMD_3225-4Pin_3.2x2.5mm, symbol Device:Crystal_GND24
- C16, C17: value 0.1uF -> 10pF; footprint Capacitor_SMD:C_0805_2012Metric -> Capacitor_SMD:C_0402_1005Metric; DK 1276-6840-1-ND -> (none); LCSC C28233 -> (none); MPN (none) -> GRM1555C1E100JA01D; Manufacturer (none) -> Murata Electronics; PARTNO CL21B104KCFNNNE -> (none)
- renumbered C17 to C1, C8 to C10, C14 to C11, C49 to C12, C15 to C13, C9 to C2, C10 to C3, C43 to C4, C7 to C5, C11 to C6, C12 to C7, C13 to C8, C48 to C9, D3 to D1, J3 to J1, J13 to J10, J13 to J11, J13 to J12, J1 to J13, J4 to J2, J14 to J5, J15 to J6, J16 to J7, J17 to J8, J12 to J9, R19 to R1, R47 to R10, R48 to R11, R23 to R12, R28 to R13, R28 to R14, R28 to R15, R28 to R16, R28 to R17, R28 to R18, R28 to R19, R17 to R2, R31 to R20, R28 to R21, R31 to R22, R28 to R23, R31 to R24, R28 to R25, R28 to R26, R28 to R27, R33 to R28, R33 to R29, R18 to R3, R33 to R30, R9 to R4, R10 to R5, R11 to R6, R12 to R7, R22 to R8, R23 to R9, TP6 to TP1, TP6 to TP2, TP6 to TP3, TP35 to TP4, TP34 to TP5, U5 to U1
Connections:
- net GND: now also C14.2, C15.2, C18.2, C19.2, C20.2, C21.2, C22.2, C23.2, C24.2, C25.2, C26.2, C27.2, C28.2, C29.2, C30.2, C31.2, C32.2, C33.2, J14.A1 (GND), J14.A12 (GND), J14.A5 (CC1), J14.B1 (GND), J14.B12 (GND), J14.B5 (CC2), J14.S1 (SHIELD), J15.2 (Pin_2), J15.MP (MountPin), SW1.1, SW1.SH1, SW1.SH2, U3.62 (VREG_PGND), U3.81 (GND), U4.4 (GND), Y1.2, Y1.4
- net at C17.1: now also R32.2, Y1.3
- net XIN: now reaches C16.1
- net XIN: now also U3.30 (XIN), Y1.1
- net VCCIO renamed +3.3v
- net VCORE renamed 1V8
- new net: C26.1, C29.1, R36.1, U3.59 (ADC_AVDD)
- new net: D2.1 (K), PTC1.2
- new net: D3.2 (A), R34.2
- new net +3V3: C23.1, C24.1, C25.1, C27.1, C28.1, C30.1, C31.1, C32.1, C33.1, R31.2, R33.2, R35.1, R36.2, U3.15 (IOVDD), U3.24 (IOVDD), U3.29 (IOVDD), U3.41 (IOVDD), U3.5 (IOVDD), U3.50 (IOVDD), U3.60 (IOVDD), U3.68 (USB_OTP_VDD), U3.69 (QSPI_IOVDD), U3.76 (IOVDD), U4.8 (VCC)
- new net 1V1: C15.1, C19.1, C21.1, C22.1, L1.1, U3.10 (DVDD), U3.32 (DVDD), U3.51 (DVDD), U3.65 (VREG_FB)
- new net QSPI_SCLK: U3.71 (QSPI_SCLK), U4.6 (CLK)
- new net QSPI_SD0: U3.72 (QSPI_SD0), U4.5 (DI(IO0))
- new net QSPI_SD1: U3.74 (QSPI_SD1), U4.2 (DO(IO1))
- new net QSPI_SD2: U3.73 (QSPI_SD2), U4.3 (IO2)
- new net QSPI_SD3: U3.70 (QSPI_SD3), U4.7 (IO3)
- new net SWCLK: J15.1 (Pin_1), U3.33 (SWCLK)
- new net SWD: J15.3 (Pin_3), U3.34 (SWD)
- new net USB_D+: J14.A6 (D+), J14.B6 (D+), R37.1
- new net USB_D-: J14.A7 (D-), J14.B7 (D-), R38.1
- new net USB_N: R38.2, U3.66 (USB_DM)
- new net USB_P: R37.2, U3.67 (USB_DP)
- new net VBUS: D2.2 (A), J14.A4 (VBUS), J14.A9 (VBUS), J14.B4 (VBUS), J14.B9 (VBUS)
- new net VIN: C14.1, C20.1, PTC1.1, U3.64 (VREG_VIN)
- new net VREG_AVDD: C18.1, R31.1, U3.61 (VREG_AVDD)
- new net VREG_LX: L1.2, U3.63 (VREG_LX)
- new net XOUT: R32.1, U3.31 (XOUT)
- new net ~{QSPI_SS}: R34.1, U3.75 (QSPI_SS), U4.1 (~{CS})
- new net ~{RESET}: R33.1, U3.35 (RUN)
- new net ~{USB_BOOT}: D3.1 (K), R35.2, SW1.2
- no-connect marks 24 -> 10
Other:
- note added: "CSn0"
- note added: "JST Debug Connector"
- note added: "MISO0"
- note added: "MISO1"
- note added: "MOSI0"
- note added: "MOSI1"
- note added: "Place R4/R5 close to RP2040"
- note added: "Raspberry Pico"
- note added: "SCK0"
- note added: "SCK1"
- note added: "SSn1"
- note added: "https://datasheets.raspberrypi.com/rp2350/hardware-design-with-rp2350.pdf"
